File: PB170/LC.sch (KiCad schematic (older format))
At the start: 7 parts

Commit message: added some labels
Parts:
- added U?: 74HC00, Package_SO:TSSOP-14_4.4x5mm_P0.65mm, symbol 74xx:74HC00
- U? (x2): value 74HC32 -> 74HC00; footprint Housings_SOIC:SOIC-14_3.9x8.7mm_Pitch1.27mm -> Package_SO:TSSOP-14_4.4x5mm_P0.65mm
- U? (x3): value 74HC08 -> 74HC00; footprint Housings_SOIC:SOIC-14_3.9x8.7mm_Pitch1.27mm -> Package_SO:TSSOP-14_4.4x5mm_P0.65mm
Connections:
- net 11: now reaches U?.10 (3B)
- net 10: now reaches U?.2 (1B)
- net at U?.5 (2B): now also U?.8
- new net 00: U?.10, U?.9
Other:
- moved on the sheet: U?A, U?B, U?C, U?D
Changed lines of the file:
@@
 $Descr A4 11693 8268
 encoding utf-8
-Sheet 4 7
+Sheet 4 6
 Title ""
 Date ""
@@
 L PB170:74HC08 U?
 U 3 1 60280058
-P 1650 1400
-F 0 "U?" H 1675 1667 50  0000 C CNN
-F 1 "74HC08" H 1675 1576 50  0000 C CNN
-F 2 "Housings_SOIC:SOIC-14_3.9x8.7mm_Pitch1.27mm" H 1650 1400 50  0001 C CNN
-F 3 "https://datasheet.lcsc.com/szlcsc/Nexperia-74HC08D-653_C5593.pdf" H 1650 1400 50  0001 C CNN
-F 4 "C5593" H 1650 1400 50  0001 C CNN "LCSC"
-	3    1650 1400
+P 5350 3000
+F 0 "U?" H 5375 3267 50  0000 C CNN
+F 1 "74HC08" H 5375 3176 50  0000 C CNN
+F 2 "Housings_SOIC:SOIC-14_3.9x8.7mm_Pitch1.27mm" H 5350 3000 50  0001 C CNN
+F 3 "https://datasheet.lcsc.com/szlcsc/Nexperia-74HC08D-653_C5593.pdf" H 5350 3000 50  0001 C CNN
+F 4 "C5593" H 5350 3000 50  0001 C CNN "LCSC"
+	3    5350 3000
 	1    0    0    -1
 $EndComp
@@
 L PB170:74HC08 U?
 U 4 1 60280745
-P 1650 1900
-F 0 "U?" H 1675 2167 50  0000 C CNN
-F 1 "74HC08" H 1675 2076 50  0000 C CNN
-F 2 "Housings_SOIC:SOIC-14_3.9x8.7mm_Pitch1.27mm" H 1650 1900 50  0001 C CNN
-F 3 "https://datasheet.lcsc.com/szlcsc/Nexperia-74HC08D-653_C5593.pdf" H 1650 1900 50  0001 C CNN
-F 4 "C5593" H 1650 1900 50  0001 C CNN "LCSC"
-	4    1650 1900
+P 5350 3500
+F 0 "U?" H 5375 3767 50  0000 C CNN
+F 1 "74HC00" H 5375 3676 50  0000 C CNN
+F 2 "Package_SO:TSSOP-14_4.4x5mm_P0.65mm" H 5350 3500 50  0001 C CNN
+F 3 "https://datasheet.lcsc.com/szlcsc/Texas-Instruments-TI-SN74HC00PWR_C6807.pdf" H 5350 3500 50  0001 C CNN
+F 4 "C5593" H 5350 3500 50  0001 C CNN "LCSC"
+	4    5350 3500
 	1    0    0    -1
 $EndComp
@@
 L PB170:74HC08 U?
 U 1 1 60280E2E
-P 1650 2400
-F 0 "U?" H 1675 2667 50  0000 C CNN
-F 1 "74HC08" H 1675 2576 50  0000 C CNN
-F 2 "Housings_SOIC:SOIC-14_3.9x8.7mm_Pitch1.27mm" H 1650 2400 50  0001 C CNN
-F 3 "https://datasheet.lcsc.com/szlcsc/Nexperia-74HC08D-653_C5593.pdf" H 1650 2400 50  0001 C CNN
-F 4 "C5593" H 1650 2400 50  0001 C CNN "LCSC"
-	1    1650 2400
+P 5350 4000
+F 0 "U?" H 5375 4267 50  0000 C CNN
+F 1 "74HC00" H 5375 4176 50  0000 C CNN
+F 2 "Package_SO:TSSOP-14_4.4x5mm_P0.65mm" H 5350 4000 50  0001 C CNN
+F 3 "https://datasheet.lcsc.com/szlcsc/Texas-Instruments-TI-SN74HC00PWR_C6807.pdf" H 5350 4000 50  0001 C CNN
+F 4 "C5593" H 5350 4000 50  0001 C CNN "LCSC"
+	1    5350 4000
 	1    0    0    -1
 $EndComp
@@
 L PB170:74HC08 U?
 U 2 1 60281A2A
-P 1650 2850
-F 0 "U?" H 1675 3117 50  0000 C CNN
-F 1 "74HC08" H 1675 3026 50  0000 C CNN
-F 2 "Housings_SOIC:SOIC-14_3.9x8.7mm_Pitch1.27mm" H 1650 2850 50  0001 C CNN
-F 3 "https://datasheet.lcsc.com/szlcsc/Nexperia-74HC08D-653_C5593.pdf" H 1650 2850 50  0001 C CNN
-F 4 "C5593" H 1650 2850 50  0001 C CNN "LCSC"
-	2    1650 2850
+P 5350 4450
+F 0 "U?" H 5375 4717 50  0000 C CNN
+F 1 "74HC00" H 5375 4626 50  0000 C CNN
+F 2 "Package_SO:TSSOP-14_4.4x5mm_P0.65mm" H 5350 4450 50  0001 C CNN
+F 3 "https://datasheet.lcsc.com/szlcsc/Texas-Instruments-TI-SN74HC00PWR_C6807.pdf" H 5350 4450 50  0001 C CNN
+F 4 "C5593" H 5350 4450 50  0001 C CNN "LCSC"
+	2    5350 4450
 	1    0    0    -1
 $EndComp
@@
 L PB170:74HC32 U?
 U 1 1 6025D6DD
-P 2700 1700
-F 0 "U?" H 2675 1975 50  0000 C CNN
-F 1 "74HC32" H 2675 1884 50  0000 C CNN
-F 2 "Housings_SOIC:SOIC-14_3.9x8.7mm_Pitch1.27mm" H 2150 1900 50  0001 C CNN
-F 3 "https://datasheet.lcsc.com/szlcsc/Nexperia-74HC32D-653_C5632.pdf" H 2150 1900 50  0001 C CNN
-F 4 "C5632" H 2700 1700 50  0001 C CNN "LCSC"
-	1    2700 1700
+P 6400 3300
+F 0 "U?" H 6375 3575 50  0000 C CNN
+F 1 "74HC00" H 6375 3484 50  0000 C CNN
+F 2 "Package_SO:TSSOP-14_4.4x5mm_P0.65mm" H 5850 3500 50  0001 C CNN
+F 3 "https://datasheet.lcsc.com/szlcsc/Texas-Instruments-TI-SN74HC00PWR_C6807.pdf" H 5850 3500 50  0001 C CNN
+F 4 "C5632" H 6400 3300 50  0001 C CNN "LCSC"
+	1    6400 3300
 	1    0    0    -1
 $EndComp
@@
 L PB170:74HC32 U?
 U 2 1 6025E1D5
-P 2700 2600
-F 0 "U?" H 2675 2875 50  0000 C CNN
-F 1 "74HC32" H 2675 2784 50  0000 C CNN
-F 2 "Housings_SOIC:SOIC-14_3.9x8.7mm_Pitch1.27mm" H 2150 2800 50  0001 C CNN
-F 3 "https://datasheet.lcsc.com/szlcsc/Nexperia-74HC32D-653_C5632.pdf" H 2150 2800 50  0001 C CNN
-F 4 "C5632" H 2700 2600 50  0001 C CNN "LCSC"
-	2    2700 2600
+P 6400 4200
+F 0 "U?" H 6375 4475 50  0000 C CNN
+F 1 "74HC00" H 6375 4384 50  0000 C CNN
+F 2 "Package_SO:TSSOP-14_4.4x5mm_P0.65mm" H 5850 4400 50  0001 C CNN
+F 3 "https://datasheet.lcsc.com/szlcsc/Texas-Instruments-TI-SN74HC00PWR_C6807.pdf" H 5850 4400 50  0001 C CNN
+F 4 "C5632" H 6400 4200 50  0001 C CNN "LCSC"
+	2    6400 4200
 	1    0    0    -1
 $EndComp
@@
 L PB170:74HC32 U?
 U 3 1 6025EF5C
-P 3450 2150
-F 0 "U?" H 3425 2425 50  0000 C CNN
-F 1 "74HC32" H 3425 2334 50  0000 C CNN
-F 2 "Housings_SOIC:SOIC-14_3.9x8.7mm_Pitch1.27mm" H 2900 2350 50  0001 C CNN
-F 3 "https://datasheet.lcsc.com/szlcsc/Nexperia-74HC32D-653_C5632.pdf" H 2900 2350 50  0001 C CNN
-F 4 "C5632" H 3450 2150 50  0001 C CNN "LCSC"
-	3    3450 2150
+P 7150 3750
+F 0 "U?" H 7125 4025 50  0000 C CNN
+F 1 "74HC32" H 7125 3934 50  0000 C CNN
+F 2 "Housings_SOIC:SOIC-14_3.9x8.7mm_Pitch1.27mm" H 6600 3950 50  0001 C CNN
+F 3 "https://datasheet.lcsc.com/szlcsc/Nexperia-74HC32D-653_C5632.pdf" H 6600 3950 50  0001 C CNN
+F 4 "C5632" H 7150 3750 50  0001 C CNN "LCSC"
+	3    7150 3750
 	1    0    0    -1
 $EndComp
 Wire Wire Line
-	1950 1400 2300 1400
+	5650 3000 6000 3000
 Wire Wire Line
-	2300 1400 2300 1650
+	6000 3000 6000 3250
 Wire Wire Line
-	2300 1650 2450 1650
+	6000 3250 6150 3250
 Wire Wire Line
-	1950 1900 2300 1900
+	5650 3500 6000 3500
 Wire Wire Line
-	2300 1900 2300 1750
+	6000 3500 6000 3350
 Wire Wire Line
-	2300 1750 2450 1750
+	6000 3350 6150 3350
 Wire Wire Line
-	1950 2400 2300 2400
+	5650 4000 6000 4000
 Wire Wire Line
-	2300 2400 2300 2550
+	6000 4000 6000 4150
 Wire Wire Line
-	2300 2550 2450 2550
+	6000 4150 6150 4150
 Wire Wire Line
-	1950 2850 2300 2850
+	5650 4450 6000 4450
 Wire Wire Line
-	2300 2850 2300 2650
+	6000 4450 6000 4250
 Wire Wire Line
-	2300 2650 2450 2650
+	6000 4250 6150 4250
 Wire Wire Line
-	2900 1700 3100 1700
+	6600 3300 6800 3300
 Wire Wire Line
-	3100 1700 3100 2100
+	6800 3300 6800 3700
 Wire Wire Line
-	3100 2100 3200 2100
+	6800 3700 6900 3700
 Wire Wire Line
-	2900 2600 3100 2600
+	6600 4200 6800 4200
 Wire Wire Line
-	3100 2600 3100 2200
+	6800 4200 6800 3800
 Wire Wire Line
-	3100 2200 3200 2200
-Text GLabel 3650 2150 2    50   Output ~ 0
+	6800 3800 6900 3800
+Text GLabel 7350 3750 2    50   Output ~ 0
 LC
-Text GLabel 1400 1350 0    50   Input ~ 0
+Text GLabel 5100 2950 0    50   Input ~ 0
 Q0
-Text GLabel 1400 1850 0    50   Input ~ 0
+Text GLabel 5100 3450 0    50   Input ~ 0
 Q2
-Text GLabel 1400 1950 0    50   Input ~ 0
+Text GLabel 5100 3550 0    50   Input ~ 0
 !I0
-Text GLabel 1400 2350 0    50   Input ~ 0
+Text GLabel 5100 3950 0    50   Input ~ 0
 Q3
-Text GLabel 1400 2800 0    50   Input ~ 0
+Text GLabel 5100 4400 0    50   Input ~ 0
 Q4
+Text GLabel 5100 3050 0    50   Input ~ 0
+11
+Text GLabel 5100 4050 0    50   Input ~ 0
+10
+$Comp
+L 74xx:74HC00 U?
+U 3 1 6028EBF4
+P 4550 4500
+AR Path="/6026D736/6028EBF4" Ref="U?"  Part="1"
+AR Path="/6026F362/6028EBF4" Ref="U?"  Part="3"
+F 0 "U?" H 4550 4825 50  0000 C CNN
+F 1 "74HC00" H 4550 4734 50  0000 C CNN
+F 2 "Package_SO:TSSOP-14_4.4x5mm_P0.65mm" H 4550 4500 50  0001 C CNN
+F 3 "https://datasheet.lcsc.com/szlcsc/Texas-Instruments-TI-SN74HC00PWR_C6807.pdf" H 4550 4500 50  0001 C CNN
+F 4 "C6807" H 4550 4500 50  0001 C CNN "LCSC"
+	3    4550 4500
+	1    0    0    -1
+$EndComp
+Wire Wire Line
+	5100 4500 4850 4500
+Wire Wire Line
+	4250 4400 4150 4400
+Wire Wire Line
+	4150 4400 4150 4500
+Wire Wire Line
+	4150 4600 4250 4600
+Wire Wire Line
+	4150 4500 4050 4500
+Connection ~ 4150 4500
+Wire Wire Line
+	4150 4500 4150 4600
+Text GLabel 4050 4500 0    50   Input ~ 0
+00
 $EndSCHEMATC
