File: PB170/LC.sch (KiCad schematic (older format))
At the start: 8 parts

Commit message: added LEDs, mby we could try to start routing
Parts:
- added U?: 74HC00, Package_SO:TSSOP-14_4.4x5mm_P0.65mm, symbol PB170:74HC08
- U?: value 74HC32 -> 74HC00; footprint Housings_SOIC:SOIC-14_3.9x8.7mm_Pitch1.27mm -> Package_SO:TSSOP-14_4.4x5mm_P0.65mm
- U?: value 74HC08 -> 74HC00; footprint Housings_SOIC:SOIC-14_3.9x8.7mm_Pitch1.27mm -> Package_SO:TSSOP-14_4.4x5mm_P0.65mm
Connections:
- net LC: now also U?.11 (4Y); no longer U?.8 (3Y)
- net at U?.8 (3Y): now also U?.4 (2A); no longer U?.1 (1A)
- net at U?.11 (4Y): now also U?.5 (2B); no longer U?.2 (1B)
- net at U?.3 (1Y): now also U?.9 (3A); no longer U?.4 (2A)
- net at U?.6 (2Y): now also U?.10 (3B); no longer U?.5 (2B)
- new net: U?.12 (4A), U?.6 (2Y)
- new net: U?.13 (4B), U?.8 (3Y)
- new net +5V: U?.14 (VCC)
- new net GND: U?.7 (GND)
Changed lines of the file:
@@
 P 5350 3000
 F 0 "U?" H 5375 3267 50  0000 C CNN
-F 1 "74HC08" H 5375 3176 50  0000 C CNN
-F 2 "Housings_SOIC:SOIC-14_3.9x8.7mm_Pitch1.27mm" H 5350 3000 50  0001 C CNN
-F 3 "https://datasheet.lcsc.com/szlcsc/Nexperia-74HC08D-653_C5593.pdf" H 5350 3000 50  0001 C CNN
+F 1 "74HC00" H 5375 3176 50  0000 C CNN
+F 2 "Package_SO:TSSOP-14_4.4x5mm_P0.65mm" H 5350 3000 50  0001 C CNN
+F 3 "https://datasheet.lcsc.com/szlcsc/Texas-Instruments-TI-SN74HC00PWR_C6807.pdf" H 5350 3000 50  0001 C CNN
 F 4 "C5593" H 5350 3000 50  0001 C CNN "LCSC"
 	3    5350 3000
@@
 $Comp
 L PB170:74HC32 U?
-U 1 1 6025D6DD
+U 2 1 6025D6DD
 P 6400 3300
 F 0 "U?" H 6375 3575 50  0000 C CNN
@@
 F 3 "https://datasheet.lcsc.com/szlcsc/Texas-Instruments-TI-SN74HC00PWR_C6807.pdf" H 5850 3500 50  0001 C CNN
 F 4 "C5632" H 6400 3300 50  0001 C CNN "LCSC"
-	1    6400 3300
+	2    6400 3300
 	1    0    0    -1
 $EndComp
 $Comp
 L PB170:74HC32 U?
-U 2 1 6025E1D5
+U 3 1 6025E1D5
 P 6400 4200
 F 0 "U?" H 6375 4475 50  0000 C CNN
@@
 F 3 "https://datasheet.lcsc.com/szlcsc/Texas-Instruments-TI-SN74HC00PWR_C6807.pdf" H 5850 4400 50  0001 C CNN
 F 4 "C5632" H 6400 4200 50  0001 C CNN "LCSC"
-	2    6400 4200
+	3    6400 4200
 	1    0    0    -1
 $EndComp
 $Comp
 L PB170:74HC32 U?
-U 3 1 6025EF5C
+U 4 1 6025EF5C
 P 7150 3750
 F 0 "U?" H 7125 4025 50  0000 C CNN
-F 1 "74HC32" H 7125 3934 50  0000 C CNN
-F 2 "Housings_SOIC:SOIC-14_3.9x8.7mm_Pitch1.27mm" H 6600 3950 50  0001 C CNN
-F 3 "https://datasheet.lcsc.com/szlcsc/Nexperia-74HC32D-653_C5632.pdf" H 6600 3950 50  0001 C CNN
+F 1 "74HC00" H 7125 3934 50  0000 C CNN
+F 2 "Package_SO:TSSOP-14_4.4x5mm_P0.65mm" H 6600 3950 50  0001 C CNN
+F 3 "https://datasheet.lcsc.com/szlcsc/Texas-Instruments-TI-SN74HC00PWR_C6807.pdf" H 6600 3950 50  0001 C CNN
 F 4 "C5632" H 7150 3750 50  0001 C CNN "LCSC"
-	3    7150 3750
+	4    7150 3750
 	1    0    0    -1
 $EndComp
@@
 Text GLabel 4050 4500 0    50   Input ~ 0
 00
+$Comp
+L PB170:74HC08 U?
+U 5 1 60279967
+P 8600 3750
+AR Path="/6026D736/60279967" Ref="U?"  Part="5"
+AR Path="/6026F362/60279967" Ref="U?"  Part="5"
+F 0 "U?" H 8830 3796 50  0000 L CNN
+F 1 "74HC00" H 8830 3705 50  0000 L CNN
+F 2 "Package_SO:TSSOP-14_4.4x5mm_P0.65mm" H 8600 3750 50  0001 C CNN
+F 3 "https://datasheet.lcsc.com/szlcsc/Texas-Instruments-TI-SN74HC00PWR_C6807.pdf" H 8600 3750 50  0001 C CNN
+F 4 "C5593" H 8600 3750 50  0001 C CNN "LCSC"
+	5    8600 3750
+	1    0    0    -1
+$EndComp
+$Comp
+L power:GND #PWR?
+U 1 1 6027996D
+P 8600 4250
+AR Path="/6026D736/6027996D" Ref="#PWR?"  Part="1"
+AR Path="/6026F362/6027996D" Ref="#PWR?"  Part="1"
+F 0 "#PWR?" H 8600 4000 50  0001 C CNN
+F 1 "GND" H 8605 4077 50  0000 C CNN
+F 2 "" H 8600 4250 50  0001 C CNN
+F 3 "" H 8600 4250 50  0001 C CNN
+	1    8600 4250
+	1    0    0    -1
+$EndComp
+$Comp
+L power:+5V #PWR?
+U 1 1 60279973
+P 8600 3250
+AR Path="/6026D736/60279973" Ref="#PWR?"  Part="1"
+AR Path="/6026F362/60279973" Ref="#PWR?"  Part="1"
+F 0 "#PWR?" H 8600 3100 50  0001 C CNN
+F 1 "+5V" H 8615 3423 50  0000 C CNN
+F 2 "" H 8600 3250 50  0001 C CNN
+F 3 "" H 8600 3250 50  0001 C CNN
+	1    8600 3250
+	1    0    0    -1
+$EndComp
 $EndSCHEMATC
