File: PB170/PB170.sch (KiCad schematic (older format))
At the start: 50 parts, among them J1 USB_C_Receptacle_USB2.0-Conne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, J2 USB_B_Micro, Q1 P-MOSFET-MLP_HS, Q2 BC817, SW1 SW_MEC_5E, SW2 SW_MEC_5E

Commit message: PB170.sch change
Parts:
- added U?: 74HC08, Housings_SOIC:SOIC-14_3.9x8.7mm_Pitch1.27mm, symbol PB170:74HC08
- added U? (x4): 74HC74, Package_SO:TSSOP-14_4.4x5mm_P0.65mm, symbol PB170:74HC08
- added U? (x3): 74HC74, Package_SO:TSSOP-14_4.4x5mm_P0.65mm, symbol 74xx:74HC74
Connections:
- net +5V: now also U?.1 (~R), U?.10 (~S), U?.14 (VCC), U?.14 (VCC), U?.4 (~S)
- net CLOCK: now also U?.3 (C)
- net GND: now also U?.7 (GND), U?.7 (GND)
- net SET: now also U?.13 (~R)
- new net !I0: U?.10 (3B), U?.11 (C), U?.2 (1B), U?.2 (D), U?.6 (~Q)
- new net !I1: U?.1 (1A), U?.12 (D), U?.4 (2A), U?.8 (~Q)
- new net 00: U?.3 (1Y)
- new net 01: U?.6 (2Y)
- new net 10: U?.8 (3Y)
- new net 11: U?.11 (4Y)
- new net I0: U?.13 (4B), U?.5 (2B), U?.5 (Q)
- new net I1: U?.12 (4A), U?.9 (3A), U?.9 (Q)
Other:
- note added: "2-bit counter"
- note removed: "No idea what to do with the unused one."
- moved on the sheet: U?C

Commit message: added some labels
Parts:
- removed C3, C4: 10uF, Capacitors_SMD:C_0805, symbol Device:C
- removed D2, D3: LED yellow, LEDs:LED_0603, symbol Device:LED
- removed D4: LED green, LEDs:LED_0603, symbol Device:LED
- removed D5: LED blue, LEDs:LED_0603, symbol Device:LED
- removed D6: LED white, LEDs:LED_0603, symbol Device:LED
- removed Q2: BC817, TO_SOT_Packages_SMD:SOT-23, symbol Transistor_BJT:BC817
- removed R12, R7: 220R, Resistors_SMD:R_0603, symbol Device:R
- removed R2, R3, R6: 180R, Resistors_SMD:R_0603, symbol Device:R
- removed R4, R5: 10k, Resistors_SMD:R_0603, symbol Device:R
- removed R8: 130R, Resistors_SMD:R_0603, symbol Device:R
- removed SW1, SW2: SW_MEC_5E, PB170:TactileSwitch_C381064, symbol Switch:SW_MEC_5E
- added C?: 10uF, Capacitors_SMD:C_0805, symbol Device:C
- added R?: 10k, Resistors_SMD:R_0603, symbol Device:R
- added SW?: SW_MEC_5E, PB170:TactileSwitch_C381064, symbol Switch:SW_MEC_5E
Connections:
- net +5V: now also C?.2, SW?.1, SW?.2
- net CLOCK: no longer U?.3 (C)
- net GND: now also R?.2
- new net MODE: C?.1, R?.1, SW?.3 (K), SW?.4 (A), U?.3 (C)
Other:
- note added: "Input combinations"
- note added: "MODE Button"
- note removed: "XOR using 4 NANDs"
- moved on the sheet: U?A, U?B, U?C, U?D, U?E

Commit message: 12-02-2021 Martin
Parts:
- added D? (x5): LED red, LEDs:LED_0603, symbol Device:LED
- added R? (x5): 220R, Resistors_SMD:R_0603, symbol Device:R
Connections:
- net GND: now also D?.1 (K), D?.1 (K), D?.1 (K), D?.1 (K), D?.1 (K)
- new net: D?.2 (A), R?.2 (x5)
- new net LA: R?.1
- new net LB: R?.1
- new net LC: R?.1
- new net LD: R?.1
- new net LE: R?.1
Other:
- moved on the sheet: D1, R1
Changed lines of the file:
@@
 L Device:R R1
 U 1 1 5FCE05A1
-P 1400 3550
-F 0 "R1" H 1470 3596 50  0000 L CNN
-F 1 "220R" H 1470 3505 50  0000 L CNN
-F 2 "Resistors_SMD:R_0603" V 1330 3550 50  0001 C CNN
-F 3 "https://datasheet.lcsc.com/szlcsc/Uniroyal-Elec-0603WAF2200T5E_C22962.pdf" H 1400 3550 50  0001 C CNN
-F 4 "C22962" H 1400 3550 50  0001 C CNN "LCSC"
-	1    1400 3550
+P 1450 3650
+F 0 "R1" H 1520 3696 50  0000 L CNN
+F 1 "220R" H 1520 3605 50  0000 L CNN
+F 2 "Resistors_SMD:R_0603" V 1380 3650 50  0001 C CNN
+F 3 "https://datasheet.lcsc.com/szlcsc/Uniroyal-Elec-0603WAF2200T5E_C22962.pdf" H 1450 3650 50  0001 C CNN
+F 4 "C22962" H 1450 3650 50  0001 C CNN "LCSC"
+	1    1450 3650
 	1    0    0    -1
 $EndComp
@@
 L Device:LED D1
 U 1 1 5FCE0D28
-P 1400 3850
-F 0 "D1" V 1439 3733 50  0000 R CNN
-F 1 "LED red" V 1348 3733 50  0000 R CNN
-F 2 "LEDs:LED_0603" H 1400 3850 50  0001 C CNN
-F 3 "https://datasheet.lcsc.com/szlcsc/Hubei-KENTO-Elec-KT-0603R_C2286.pdf" H 1400 3850 50  0001 C CNN
-F 4 "C2286" V 1400 3850 50  0001 C CNN "LCSC"
-	1    1400 3850
+P 1450 3950
+F 0 "D1" V 1489 3833 50  0000 R CNN
+F 1 "LED red" V 1398 3833 50  0000 R CNN
+F 2 "LEDs:LED_0603" H 1450 3950 50  0001 C CNN
+F 3 "https://datasheet.lcsc.com/szlcsc/Hubei-KENTO-Elec-KT-0603R_C2286.pdf" H 1450 3950 50  0001 C CNN
+F 4 "C2286" V 1450 3950 50  0001 C CNN "LCSC"
+	1    1450 3950
 	0    -1   -1   0
 $EndComp
@@
 L power:GND #PWR0106
 U 1 1 5FD0AF6E
-P 1400 4000
-F 0 "#PWR0106" H 1400 3750 50  0001 C CNN
-F 1 "GND" H 1405 3827 50  0000 C CNN
-F 2 "" H 1400 4000 50  0001 C CNN
-F 3 "" H 1400 4000 50  0001 C CNN
-	1    1400 4000
+P 1450 4100
+F 0 "#PWR0106" H 1450 3850 50  0001 C CNN
+F 1 "GND" H 1455 3927 50  0000 C CNN
+F 2 "" H 1450 4100 50  0001 C CNN
+F 3 "" H 1450 4100 50  0001 C CNN
+	1    1450 4100
 	1    0    0    -1
 $EndComp
@@
 L power:+5V #PWR0107
 U 1 1 5FD0B607
-P 1400 3400
-F 0 "#PWR0107" H 1400 3250 50  0001 C CNN
-F 1 "+5V" H 1415 3573 50  0000 C CNN
-F 2 "" H 1400 3400 50  0001 C CNN
-F 3 "" H 1400 3400 50  0001 C CNN
-	1    1400 3400
+P 1450 3500
+F 0 "#PWR0107" H 1450 3350 50  0001 C CNN
+F 1 "+5V" H 1465 3673 50  0000 C CNN
+F 2 "" H 1450 3500 50  0001 C CNN
+F 3 "" H 1450 3500 50  0001 C CNN
+	1    1450 3500
 	1    0    0    -1
 $EndComp
@@
 Text Notes 11550 3000 0    50   ~ 0
 MODE Button
+$Comp
+L Device:R R?
+U 1 1 602F22C9
+P 20300 8250
+F 0 "R?" H 20370 8296 50  0000 L CNN
+F 1 "220R" H 20370 8205 50  0000 L CNN
+F 2 "Resistors_SMD:R_0603" V 20230 8250 50  0001 C CNN
+F 3 "https://datasheet.lcsc.com/szlcsc/Uniroyal-Elec-0603WAF2200T5E_C22962.pdf" H 20300 8250 50  0001 C CNN
+F 4 "C22962" H 20300 8250 50  0001 C CNN "LCSC"
+	1    20300 8250
+	1    0    0    -1
+$EndComp
+$Comp
+L Device:LED D?
+U 1 1 602F22D0
+P 20300 8550
+F 0 "D?" V 20339 8433 50  0000 R CNN
+F 1 "LED red" V 20248 8433 50  0000 R CNN
+F 2 "LEDs:LED_0603" H 20300 8550 50  0001 C CNN
+F 3 "https://datasheet.lcsc.com/szlcsc/Hubei-KENTO-Elec-KT-0603R_C2286.pdf" H 20300 8550 50  0001 C CNN
+F 4 "C2286" V 20300 8550 50  0001 C CNN "LCSC"
+	1    20300 8550
+	0    -1   -1   0
+$EndComp
+$Comp
+L power:GND #PWR?
+U 1 1 602F22D6
+P 20300 8700
+F 0 "#PWR?" H 20300 8450 50  0001 C CNN
+F 1 "GND" H 20305 8527 50  0000 C CNN
+F 2 "" H 20300 8700 50  0001 C CNN
+F 3 "" H 20300 8700 50  0001 C CNN
+	1    20300 8700
+	1    0    0    -1
+$EndComp
+$Comp
+L Device:R R?
+U 1 1 602F5297
+P 21150 8250
+F 0 "R?" H 21220 8296 50  0000 L CNN
+F 1 "220R" H 21220 8205 50  0000 L CNN
+F 2 "Resistors_SMD:R_0603" V 21080 8250 50  0001 C CNN
+F 3 "https://datasheet.lcsc.com/szlcsc/Uniroyal-Elec-0603WAF2200T5E_C22962.pdf" H 21150 8250 50  0001 C CNN
+F 4 "C22962" H 21150 8250 50  0001 C CNN "LCSC"
+	1    21150 8250
+	1    0    0    -1
+$EndComp
+$Comp
+L Device:LED D?
+U 1 1 602F529E
+P 21150 8550
+F 0 "D?" V 21189 8433 50  0000 R CNN
+F 1 "LED red" V 21098 8433 50  0000 R CNN
+F 2 "LEDs:LED_0603" H 21150 8550 50  0001 C CNN
+F 3 "https://datasheet.lcsc.com/szlcsc/Hubei-KENTO-Elec-KT-0603R_C2286.pdf" H 21150 8550 50  0001 C CNN
+F 4 "C2286" V 21150 8550 50  0001 C CNN "LCSC"
+	1    21150 8550
+	0    -1   -1   0
+$EndComp
+$Comp
+L power:GND #PWR?
+U 1 1 602F52A4
+P 21150 8700
+F 0 "#PWR?" H 21150 8450 50  0001 C CNN
+F 1 "GND" H 21155 8527 50  0000 C CNN
+F 2 "" H 21150 8700 50  0001 C CNN
+F 3 "" H 21150 8700 50  0001 C CNN
+	1    21150 8700
+	1    0    0    -1
+$EndComp
+$Comp
+L Device:R R?
+U 1 1 602F7D3F
+P 21900 8250
+F 0 "R?" H 21970 8296 50  0000 L CNN
+F 1 "220R" H 21970 8205 50  0000 L CNN
+F 2 "Resistors_SMD:R_0603" V 21830 8250 50  0001 C CNN
+F 3 "https://datasheet.lcsc.com/szlcsc/Uniroyal-Elec-0603WAF2200T5E_C22962.pdf" H 21900 8250 50  0001 C CNN
+F 4 "C22962" H 21900 8250 50  0001 C CNN "LCSC"
+	1    21900 8250
+	1    0    0    -1
+$EndComp
+$Comp
+L Device:LED D?
+U 1 1 602F7D46
+P 21900 8550
+F 0 "D?" V 21939 8433 50  0000 R CNN
+F 1 "LED red" V 21848 8433 50  0000 R CNN
+F 2 "LEDs:LED_0603" H 21900 8550 50  0001 C CNN
+F 3 "https://datasheet.lcsc.com/szlcsc/Hubei-KENTO-Elec-KT-0603R_C2286.pdf" H 21900 8550 50  0001 C CNN
+F 4 "C2286" V 21900 8550 50  0001 C CNN "LCSC"
+	1    21900 8550
+	0    -1   -1   0
+$EndComp
+$Comp
+L power:GND #PWR?
+U 1 1 602F7D4C
+P 21900 8700
+F 0 "#PWR?" H 21900 8450 50  0001 C CNN
+F 1 "GND" H 21905 8527 50  0000 C CNN
+F 2 "" H 21900 8700 50  0001 C CNN
+F 3 "" H 21900 8700 50  0001 C CNN
+	1    21900 8700
+	1    0    0    -1
+$EndComp
+$Comp
+L Device:R R?
+U 1 1 602FEDCB
+P 19450 8250
+F 0 "R?" H 19520 8296 50  0000 L CNN
+F 1 "220R" H 19520 8205 50  0000 L CNN
+F 2 "Resistors_SMD:R_0603" V 19380 8250 50  0001 C CNN
+F 3 "https://datasheet.lcsc.com/szlcsc/Uniroyal-Elec-0603WAF2200T5E_C22962.pdf" H 19450 8250 50  0001 C CNN
+F 4 "C22962" H 19450 8250 50  0001 C CNN "LCSC"
+	1    19450 8250
+	1    0    0    -1
+$EndComp
+$Comp
+L Device:LED D?
+U 1 1 602FEDD2
+P 19450 8550
+F 0 "D?" V 19489 8433 50  0000 R CNN
+F 1 "LED red" V 19398 8433 50  0000 R CNN
+F 2 "LEDs:LED_0603" H 19450 8550 50  0001 C CNN
+F 3 "https://datasheet.lcsc.com/szlcsc/Hubei-KENTO-Elec-KT-0603R_C2286.pdf" H 19450 8550 50  0001 C CNN
+F 4 "C2286" V 19450 8550 50  0001 C CNN "LCSC"
+	1    19450 8550
+	0    -1   -1   0
+$EndComp
+$Comp
+L power:GND #PWR?
+U 1 1 602FEDD8
+P 19450 8700
+F 0 "#PWR?" H 19450 8450 50  0001 C CNN
+F 1 "GND" H 19455 8527 50  0000 C CNN
+F 2 "" H 19450 8700 50  0001 C CNN
+F 3 "" H 19450 8700 50  0001 C CNN
+	1    19450 8700
+	1    0    0    -1
+$EndComp
+$Comp
+L Device:R R?
+U 1 1 603023B3
+P 18700 8250
+F 0 "R?" H 18770 8296 50  0000 L CNN
+F 1 "220R" H 18770 8205 50  0000 L CNN
+F 2 "Resistors_SMD:R_0603" V 18630 8250 50  0001 C CNN
+F 3 "https://datasheet.lcsc.com/szlcsc/Uniroyal-Elec-0603WAF2200T5E_C22962.pdf" H 18700 8250 50  0001 C CNN
+F 4 "C22962" H 18700 8250 50  0001 C CNN "LCSC"
+	1    18700 8250
+	1    0    0    -1
+$EndComp
+$Comp
+L Device:LED D?
+U 1 1 603023BA
+P 18700 8550
+F 0 "D?" V 18739 8433 50  0000 R CNN
+F 1 "LED red" V 18648 8433 50  0000 R CNN
+F 2 "LEDs:LED_0603" H 18700 8550 50  0001 C CNN
+F 3 "https://datasheet.lcsc.com/szlcsc/Hubei-KENTO-Elec-KT-0603R_C2286.pdf" H 18700 8550 50  0001 C CNN
+F 4 "C2286" V 18700 8550 50  0001 C CNN "LCSC"
+	1    18700 8550
+	0    -1   -1   0
+$EndComp
+$Comp
+L power:GND #PWR?
+U 1 1 603023C0
+P 18700 8700
+F 0 "#PWR?" H 18700 8450 50  0001 C CNN
+F 1 "GND" H 18705 8527 50  0000 C CNN
+F 2 "" H 18700 8700 50  0001 C CNN
+F 3 "" H 18700 8700 50  0001 C CNN
+	1    18700 8700
+	1    0    0    -1
+$EndComp
+Text GLabel 18700 8100 1    50   Input ~ 0
+LA
+Text GLabel 19450 8100 1    50   Input ~ 0
+LB
+Text GLabel 20300 8100 1    50   Input ~ 0
+LC
+Text GLabel 21150 8100 1    50   Input ~ 0
+LD
+Text GLabel 21900 8100 1    50   Input ~ 0
+LE
 $EndSCHEMATC

Commit message: added LEDs, mby we could try to start routing
Parts:
- removed J1: USB_C_Receptacle_USB2.0-Connector, PB170:USB_C_Female-16Pin-HPJF, symbol PB170:USB_C_Receptacle_USB2.0-Connector
- removed R10: 220R, Resistors_SMD:R_0603, symbol Device:R
- J2: footprint PB170:USB_Micro-B_Wuerth_629105150521_CircularHoles -> PB170:MICRO-USB-SMD_MICROXNJ; LCSC (none) -> C404969
Connections:
- net GND: now also U?.10 (~S), U?.11 (C), U?.12 (D), U?.13 (~R), U?.8 (~Q), U?.9 (Q)
- no-connect marks 9 -> 5
Other:
- moved on the sheet: J2, R11
Changed lines of the file:
@@
-$EndComp
-$Comp
-L Connector:USB_B_Micro J2
-U 1 1 5FD07183
-P 3400 6200
-F 0 "J2" H 3457 6667 50  0000 C CNN
-F 1 "USB_B_Micro" H 3457 6576 50  0000 C CNN
-F 2 "PB170:USB_Micro-B_Wuerth_629105150521_CircularHoles" H 3550 6150 50  0001 C CNN
-F 3 "~" H 3550 6150 50  0001 C CNN
-	1    3400 6200
-	1    0    0    -1
 $EndComp
 $Comp
@@
 Wire Notes Line
 	950  950  950  4450
-$Comp
-L Device:R R11
-U 1 1 5FD41C51
-P 3850 6300
-F 0 "R11" H 3920 6346 50  0000 L CNN
-F 1 "220R" H 3920 6255 50  0000 L CNN
-F 2 "Resistors_SMD:R_0603" V 3780 6300 50  0001 C CNN
-F 3 "https://datasheet.lcsc.com/szlcsc/Uniroyal-Elec-0603WAF2200T5E_C22962.pdf" H 3850 6300 50  0001 C CNN
-F 4 "C22962" H 3850 6300 50  0001 C CNN "LCSC"
-	1    3850 6300
-	0    1    1    0
-$EndComp
-Wire Wire Line
-	3700 6200 4000 6200
-Wire Wire Line
-	4000 6200 4000 6300
+Wire Wire Line
+	3000 6150 3000 6250
 $Comp
 L power:GND #PWR0121
 U 1 1 5FD447F1
-P 3300 6700
-F 0 "#PWR0121" H 3300 6450 50  0001 C CNN
-F 1 "GND" H 3305 6527 50  0000 C CNN
-F 2 "" H 3300 6700 50  0001 C CNN
-F 3 "" H 3300 6700 50  0001 C CNN
-	1    3300 6700
-	1    0    0    -1
-$EndComp
-Wire Wire Line
-	3300 6700 3300 6650
-Wire Wire Line
-	3400 6600 3400 6650
-Wire Wire Line
-	3400 6650 3300 6650
-Connection ~ 3300 6650
-Wire Wire Line
-	3300 6650 3300 6600
+P 2300 6650
+F 0 "#PWR0121" H 2300 6400 50  0001 C CNN
+F 1 "GND" H 2305 6477 50  0000 C CNN
+F 2 "" H 2300 6650 50  0001 C CNN
+F 3 "" H 2300 6650 50  0001 C CNN
+	1    2300 6650
+	1    0    0    -1
+$EndComp
+Wire Wire Line
+	2300 6650 2300 6600
+Wire Wire Line
+	2400 6550 2400 6600
+Connection ~ 2300 6600
+Wire Wire Line
+	2300 6600 2300 6550
 $Comp
 L power:+5V #PWR0122
 U 1 1 5FD489FB
-P 3750 5950
-F 0 "#PWR0122" H 3750 5800 50  0001 C CNN
-F 1 "+5V" H 3765 6123 50  0000 C CNN
-F 2 "" H 3750 5950 50  0001 C CNN
-F 3 "" H 3750 5950 50  0001 C CNN
-	1    3750 5950
-	1    0    0    -1
-$EndComp
-Wire Wire Line
-	3700 6000 3750 6000
-Wire Wire Line
-	3750 6000 3750 5950
-$Comp
-L power:GND #PWR0123
-U 1 1 5FD4C7CC
-P 1350 7250
-F 0 "#PWR0123" H 1350 7000 50  0001 C CNN
-F 1 "GND" H 1355 7077 50  0000 C CNN
-F 2 "" H 1350 7250 50  0001 C CNN
-F 3 "" H 1350 7250 50  0001 C CNN
-	1    1350 7250
-	1    0    0    -1
-$EndComp
-$Comp
-L Device:R R10
-U 1 1 5FD50BFB
-P 2600 6300
-F 0 "R10" H 2670 6346 50  0000 L CNN
-F 1 "220R" H 2670 6255 50  0000 L CNN
-F 2 "Resistors_SMD:R_0603" V 2530 6300 50  0001 C CNN
-F 3 "https://datasheet.lcsc.com/szlcsc/Uniroyal-Elec-0603WAF2200T5E_C22962.pdf" H 2600 6300 50  0001 C CNN
-F 4 "C22962" H 2600 6300 50  0001 C CNN "LCSC"
-	1    2600 6300
-	-1   0    0    1
-$EndComp
-Wire Wire Line
-	2250 6150 2300 6150
-Wire Wire Line
-	2250 6450 2300 6450
-$Comp
-L power:+5V #PWR0124
-U 1 1 5FD594C3
-P 2650 5600
-F 0 "#PWR0124" H 2650 5450 50  0001 C CNN
-F 1 "+5V" H 2665 5773 50  0000 C CNN
-F 2 "" H 2650 5600 50  0001 C CNN
-F 3 "" H 2650 5600 50  0001 C CNN
-	1    2650 5600
-	1    0    0    -1
-$EndComp
+P 2750 5900
+F 0 "#PWR0122" H 2750 5750 50  0001 C CNN
+F 1 "+5V" H 2765 6073 50  0000 C CNN
+F 2 "" H 2750 5900 50  0001 C CNN
+F 3 "" H 2750 5900 50  0001 C CNN
+	1    2750 5900
+	1    0    0    -1
+$EndComp
+Wire Wire Line
+	2700 5950 2750 5950
+Wire Wire Line
+	2750 5950 2750 5900
 Wire Notes Line
 	950  5150 950  7550
@@
 Wire Notes Line
 	4150 5150 950  5150
-NoConn ~ 3700 6400
 Text Notes 950  5100 0    50   ~ 0
 USB supply
 Text Notes 950  900  0    50   ~ 0
 Power management
-$Comp
-L PB170:USB_C_Receptacle_USB2.0-Connector J1
-U 1 1 5FD02084
-P 1650 6250
-F 0 "J1" H 1757 7117 50  0000 C CNN
-F 1 "USB_C_Receptacle_USB2.0-Connector" H 1757 7026 50  0000 C CNN
-F 2 "PB170:USB_C_Female-16Pin-HPJF" H 1800 6250 50  0001 C CNN
-F 3 "" H 1800 6250 50  0001 C CNN
-	1    1650 6250
-	1    0    0    -1
-$EndComp
-Wire Wire Line
-	1350 7250 1350 7200
-Wire Wire Line
-	1650 7150 1650 7200
-Wire Wire Line
-	1650 7200 1350 7200
-Connection ~ 1350 7200
-Wire Wire Line
-	1350 7200 1350 7150
-Wire Wire Line
-	2250 5650 2650 5650
-Wire Wire Line
-	2650 5650 2650 5600
-NoConn ~ 2250 5850
-NoConn ~ 2250 5950
-NoConn ~ 2250 6750
-NoConn ~ 2250 6850
-Wire Wire Line
-	2250 6250 2300 6250
-Wire Wire Line
-	2300 6250 2300 6150
-Connection ~ 2300 6150
-Wire Wire Line
-	2300 6150 2600 6150
-Wire Wire Line
-	2250 6350 2300 6350
-Wire Wire Line
-	2300 6350 2300 6450
-Connection ~ 2300 6450
-Wire Wire Line
-	2300 6450 2600 6450
 Wire Wire Line
 	2200 2150 2300 2150
@@
 Wire Wire Line
 	15500 3800 15300 3800
-Connection ~ 15500 6050
 $Comp
 L power:GND #PWR?
 U 1 1 603E70B7
-P 15500 6750
-F 0 "#PWR?" H 15500 6500 50  0001 C CNN
-F 1 "GND" H 15505 6577 50  0000 C CNN
-F 2 "" H 15500 6750 50  0001 C CNN
-F 3 "" H 15500 6750 50  0001 C CNN
-	1    15500 6750
+P 15500 7700
+F 0 "#PWR?" H 15500 7450 50  0001 C CNN
+F 1 "GND" H 15505 7527 50  0000 C CNN
+F 2 "" H 15500 7700 50  0001 C CNN
+F 3 "" H 15500 7700 50  0001 C CNN
+	1    15500 7700
 	1    0    0    -1
 $EndComp
@@
 $EndComp
 Wire Wire Line
-	15500 5500 15500 6050
-Wire Wire Line
-	15500 6050 15500 6750
-Wire Wire Line
-	15500 5000 15500 6050
-Wire Wire Line
 	11550 6900 11550 6800
 Connection ~ 11550 6800
@@
 Text GLabel 21900 8100 1    50   Input ~ 0
 LE
+Wire Wire Line
+	2400 6600 2300 6600
+NoConn ~ 2700 6350
+Wire Wire Line
+	2700 6150 3000 6150
+$Comp
+L Device:R R11
+U 1 1 5FD41C51
+P 2850 6250
+F 0 "R11" H 2920 6296 50  0000 L CNN
+F 1 "220R" H 2920 6205 50  0000 L CNN
+F 2 "Resistors_SMD:R_0603" V 2780 6250 50  0001 C CNN
+F 3 "https://datasheet.lcsc.com/szlcsc/Uniroyal-Elec-0603WAF2200T5E_C22962.pdf" H 2850 6250 50  0001 C CNN
+F 4 "C22962" H 2850 6250 50  0001 C CNN "LCSC"
+	1    2850 6250
+	0    1    1    0
+$EndComp
+$Comp
+L Connector:USB_B_Micro J2
+U 1 1 5FD07183
+P 2400 6150
+F 0 "J2" H 2457 6617 50  0000 C CNN
+F 1 "USB_B_Micro" H 2457 6526 50  0000 C CNN
+F 2 "PB170:MICRO-USB-SMD_MICROXNJ" H 2550 6100 50  0001 C CNN
+F 3 "https://datasheet.lcsc.com/szlcsc/1912111437_SHOU-HAN-MicroXNJ_C404969.pdf" H 2550 6100 50  0001 C CNN
+F 4 "C404969" H 2400 6150 50  0001 C CNN "LCSC"
+	1    2400 6150
+	1    0    0    -1
+$EndComp
+Wire Wire Line
+	15500 5000 15500 6050
+Wire Wire Line
+	15500 6050 15500 6600
+Connection ~ 15500 6050
+Wire Wire Line
+	15300 6950 15500 6950
+Connection ~ 15500 6950
+Wire Wire Line
+	15500 6950 15500 7150
+Wire Wire Line
+	15300 7150 15500 7150
+Wire Wire Line
+	15000 6750 15000 6600
+Wire Wire Line
+	15000 6600 15500 6600
+Connection ~ 15500 6600
+Wire Wire Line
+	15500 6600 15500 6700
+Wire Wire Line
+	14700 6950 14700 6700
+Wire Wire Line
+	14700 6700 15500 6700
+Connection ~ 15500 6700
+Wire Wire Line
+	15500 6700 15500 6950
+Wire Wire Line
+	15500 7150 15500 7450
+Connection ~ 15500 7150
+Wire Wire Line
+	15000 7350 15000 7450
+Wire Wire Line
+	15000 7450 15500 7450
+Connection ~ 15500 7450
+Wire Wire Line
+	15500 7450 15500 7550
+Wire Wire Line
+	14700 7050 14700 7550
+Wire Wire Line
+	14700 7550 15500 7550
+Connection ~ 15500 7550
+Wire Wire Line
+	15500 7550 15500 7700
 $EndSCHEMATC
